File: Electronics/2023-03-01_Twin_Io_Schematic.sch (EAGLE design)
At the start: 152 parts, among them IC1 7805, IC2 LD1117S33, U1 INA317IDGKT, U10 INA317IDGKT, U11 ADS131A04IPBSR, U12 ADS131A04IPBSR, U13 INA317IDGKT, U14 INA317IDGKT, U15 INA317IDGKT, U16 STM32F105R8T6, U17 OPA325IDBVR, U2 INA317IDGKT, U3 ADS131A04IPBSR, U4 INA317IDGKT, U5 INA317IDGKT, U6 INA317IDGKT, U7 INA317IDGKT, U8 INA317IDGKT, U9 INA317IDGKT, Y1 ABM3C-16.384MHZ-D4Y-T, Y2 ABM3C-16.384MHZ-D4Y-T, Y3 ABM3C-16.384MHZ-D4Y-T

Commit message: renamed all components and created board
Parts:
- C1, C16, C22: value 33nF/C0G -> 100n
- C10, C28, C31, C34, C7: value 1uF -> 100n
- C11, C2, C29, C32, C35, C8: value 1uF -> opt
- C13, C19, C25: value opt -> 100n
- C14, C20, C26: value 33nF/C0G -> opt
- C15, C21, C27, C6: value opt -> 33nF/C0G
- C3: value 100nF -> 33nF/C0G
- C30, C33, C36, C9: value 1uF -> 33nF/C0G
- C38, C40, C42: value 33nF/C0G -> 1uF
- C39, C41, C43: value opt -> 1uF
- C4: value 330nF -> 100n
- C44, C45, C46, C47, C48, C49, C50, C51: value 100n -> 1uF
- C5: value 100nF -> opt
- C53, C66: value 100n -> 1u
- C54: value 100n -> 330nF
- C55, C57, C58: value 100n -> 100nF
- C56: value 4u7 -> 1uF
- C59: value 100n -> 10uF
- C60: value 100n -> 4u7
- C62: value 1u -> 100n
- C63: value 10n -> 100n
- C64: value 100nF -> 100n
- C65: value 10uF -> 100n
- C67: value 1u -> 10n
- JP1: device pinhead:PINHD-1X2 -> pinhead:PINHD-1X13
- JP2: device pinhead:PINHD-1X3 -> pinhead:PINHD-1X2
- JP4: device pinhead:PINHD-1X13 -> pinhead:PINHD-1X3
- U11, U12, U3: value ADS131A04IPBSR -> INA317IDGKT; device ADS131A04IPBSR:ADS131A04IPBSR -> INA317IDGKT:INA317IDGKT
- U13, U14, U15: value INA317IDGKT -> ADS131A04IPBSR; device INA317IDGKT:INA317IDGKT -> ADS131A04IPBSR:ADS131A04IPBSR
- U16: value STM32F105R8T6 -> OPA325IDBVR; device STM32F105R8T6:STM32F105R8T6 -> OPA325IDBVR:OPA325IDBVR
- U17: value OPA325IDBVR -> STM32F105R8T6; device OPA325IDBVR:OPA325IDBVR -> STM32F105R8T6:STM32F105R8T6
Connections:
- removed net N$37 (its old number): C25.1, U9.VOUT
- new net N$33: C20.1, U7.VOUT
- net 2V5: now also JP1.13, U11.-, U11.REF, U12.-, U12.REF, U13.AIN1N, U13.AIN2N, U13.AIN3N, U13.AIN4N, U14.AIN1N, U14.AIN2N, U14.AIN3N, U14.AIN4N, U15.AIN1N, U15.AIN2N, U15.AIN3N, U15.AIN4N, U16.-IN, U16.OUT, U3.-, U3.REF; no longer JP4.13, U11.AIN1N, U11.AIN2N, U11.AIN3N, U11.AIN4N, U12.AIN1N, U12.AIN2N, U12.AIN3N, U12.AIN4N, U13.-, U13.REF, U14.-, U14.REF, U15.-, U15.REF, U17.-IN, U17.OUT, U3.AIN1N, U3.AIN2N, U3.AIN3N, U3.AIN4N
- net 3V3: now also C38.2, C43.2, C48.2, C52.1, C64.1, C67.1, R38.2, R46.1, U13.!RESET, U13.IOVDD_15, U13.IOVDD_29, U13.RESV, U14.!RESET, U14.IOVDD_15, U14.IOVDD_29, U14.RESV, U15.!RESET, U15.IOVDD_15, U15.IOVDD_29, U15.RESV, U16.V+, U17.VBAT, U17.VDDA, U17.VDD_1, U17.VDD_2, U17.VDD_3, U17.VDD_4; no longer C10.2, C30.2, C35.2, C56.1, C57.1, C58.1, R41.2, R44.1, U11.!RESET, U11.IOVDD_15, U11.IOVDD_29, U11.RESV, U12.!RESET, U12.IOVDD_15, U12.IOVDD_29, U12.RESV, U16.VBAT, U16.VDDA, U16.VDD_1, U16.VDD_2, U16.VDD_3, U16.VDD_4, U17.V+, U3.!RESET, U3.IOVDD_15, U3.IOVDD_29, U3.RESV
- net 5V: now also C1.1, C10.1, C13.1, C16.1, C19.1, C22.1, C37.2, C4.1, C42.2, C47.2, C7.1, R43.2, U11.V+, U12.V+, U13.AVDD, U14.AVDD, U15.AVDD, U3.V+; no longer C29.2, C34.2, C44.1, C49.1, C5.1, C50.1, C51.1, C52.1, C53.1, C54.1, C9.2, R46.2, U11.AVDD, U12.AVDD, U13.V+, U14.V+, U15.V+, U3.AVDD
- net 9V: now also C54.1, C56.1, C57.1, C58.1; no longer C2.1, C3.1, C4.1, C64.1
- net ADC0: now also C3.1, U13.AIN1P; no longer C1.1, U3.AIN1P
- net ADC0_CS: now also U17.PC6; no longer U16.PC6
- net ADC0_DONE: now also U13.!DONE, U17.PC0; no longer U16.PC0, U3.!DONE
- net ADC0_DRDY: now also U13.!DRDY, U17.PC1; no longer U16.PC1, U3.!DRDY
- net ADC1: now also C6.1, U13.AIN2P; no longer C12.1, U3.AIN2P
- net ADC10: now also C33.1, U15.AIN3P; no longer C40.1, U12.AIN3P
- net ADC11: now also C36.1, U15.AIN4P; no longer C42.1, U12.AIN4P
- net ADC1_CS: now also U14.!CS, U17.PC7; no longer U11.!CS, U16.PC7
- net ADC1_DONE: now also U14.!DONE, U17.PC2; no longer U11.!DONE, U16.PC2
- net ADC1_DRDY: now also U14.!DRDY, U17.PC3; no longer U11.!DRDY, U16.PC3
- net ADC2: now also C9.1, U13.AIN3P; no longer C14.1, U3.AIN3P
- net ADC2_CS: now also U15.!CS, U17.PC8; no longer U12.!CS, U16.PC8
- net ADC2_DONE: now also U15.!DONE, U17.PC4; no longer U12.!DONE, U16.PC4
- net ADC2_DRDY: now also U15.!DRDY, U17.PC5; no longer U12.!DRDY, U16.PC5
- net ADC3: now also C12.1, U13.AIN4P; no longer C16.1, U3.AIN4P
- net ADC4: now also C15.1, U14.AIN1P; no longer C18.1, U11.AIN1P
- net ADC5: now also C18.1, U14.AIN2P; no longer C20.1, U11.AIN2P
- net ADC6: now also C21.1, U14.AIN3P; no longer C22.1, U11.AIN3P
- net ADC7: now also U14.AIN4P; no longer U11.AIN4P
- net ADC8: now also C27.1, U15.AIN1P; no longer C26.1, U12.AIN1P
- net ADC9: now also C30.1, U15.AIN2P; no longer C38.1, U12.AIN2P
- net ADC_CS: now also U13.!CS; no longer U3.!CS
- net ADC_DIN: now also U13.DIN, U14.DIN, U15.DIN, U17.PA7; no longer U11.DIN, U12.DIN, U16.PA7, U3.DIN
- net ADC_DOUT: now also U13.DOUT, U14.DOUT, U15.DOUT, U17.PA6; no longer U11.DOUT, U12.DOUT, U16.PA6, U3.DOUT
- net ADC_MODE_0: now also R40.2, U13.M0, U14.M0, U15.M0; no longer R38.2, U11.M0, U12.M0, U3.M0
- net ADC_MODE_1: now also R38.1, R41.2, U13.M1, U14.M1, U15.M1; no longer R39.1, R40.2, U11.M1, U12.M1, U3.M1
- net ADC_MODE_2: now also R39.1, U13.M2, U14.M2, U15.M2; no longer R41.1, U11.M2, U12.M2, U3.M2
- net ADC_SCLK: now also U13.SCLK, U14.SCLK, U15.SCLK, U17.PA5; no longer U11.SCLK, U12.SCLK, U16.PA5, U3.SCLK
- net GND: now also C10.2, C13.2, C15.2, C19.2, C21.2, C25.2, C27.2, C30.2, C31.2, C34.2, C36.2, C38.1, C39.1, C40.1, C41.2, C42.1, C43.1, C44.1, C45.1, C47.1, C48.1, C49.1, C50.1, C53.1, C6.2, C67.2, C9.2, JP4.1, R41.1, R44.1, U11.V-, U12.V-, U13.AVSS, U13.GND, U13.REFN, U13.VNCP, U14.AVSS, U14.GND, U14.REFN, U14.VNCP, U15.AVSS, U15.GND, U15.REFN, U15.VNCP, U16.V-, U17.VSSA, U17.VSS_1, U17.VSS_2, U17.VSS_3, U17.VSS_4, U3.V-; no longer C10.1, C11.1, C14.2, C2.2, C20.2, C26.2, C29.1, C30.1, C31.1, C32.1, C34.1, C35.1, C36.1, C38.2, C40.2, C42.2, C44.2, C45.2, C47.2, C48.2, C49.2, C5.2, C50.2, C53.2, C67.1, C8.1, C9.1, JP1.1, R38.1, R43.1, U11.AVSS, U11.GND, U11.REFN, U11.VNCP, U12.AVSS, U12.GND, U12.REFN, U12.VNCP, U13.V-, U14.V-, U15.V-, U16.VSSA, U16.VSS_1, U16.VSS_2, U16.VSS_3, U16.VSS_4, U17.V-, U3.AVSS, U3.GND, U3.REFN, U3.VNCP
- net LEAD0: now also JP1.12; no longer JP4.12
- net LEAD1: now also JP1.11; no longer JP4.11
- net LEAD10: now also JP1.2, U11.+; no longer JP4.2, U14.+
- net LEAD11: now also JP1.1, U12.+; no longer JP4.1, U15.+
- net LEAD2: now also JP1.10, U3.+; no longer JP4.10, U4.+
- net LEAD3: now also JP1.9, U4.+; no longer JP4.9, U5.+
- net LEAD4: now also JP1.8, U5.+; no longer JP4.8, U6.+
- net LEAD5: now also JP1.7, U6.+; no longer JP4.7, U7.+
- net LEAD6: now also JP1.6, U7.+; no longer JP4.6, U8.+
- net LEAD7: now also JP1.5, U8.+; no longer JP4.5, U9.+
- net LEAD8: now also JP1.4, U9.+; no longer JP4.4, U10.+
- net LEAD9: now also JP1.3, U10.+; no longer JP4.3, U13.+
- net LED0: now also U17.PB0; no longer U16.PB0
- net LED1: now also U17.PB1; no longer U16.PB1
- net LED2: now also U17.PB2; no longer U16.PB2
- net N$10: now also C39.2, U13.REFEXT; no longer C11.2, U3.REFEXT
- net N$13: now also C5.1; no longer C13.1
- net N$14: now also C5.2; no longer C13.2
- net N$15: now also U3.RG1; no longer U4.RG1
- net N$16: now also U3.RG2; no longer U4.RG2
- net N$17: now also C8.1, U3.VOUT; no longer C15.1, U4.VOUT
- net N$18: now also C8.2; no longer C15.2
- net N$19: now also U4.RG1; no longer U5.RG1
- net N$20: now also U4.RG2; no longer U5.RG2
- net N$21: now also C11.1, U4.VOUT; no longer C17.1, U5.VOUT
- net N$22: now also C11.2; no longer C17.2
- net N$23: now also U5.RG1; no longer U6.RG1
- net N$24: now also U5.RG2; no longer U6.RG2
- net N$25: now also C14.1, U5.VOUT; no longer C19.1, U6.VOUT
- net N$26: now also C14.2; no longer C19.2
- net N$27: now also U6.RG1; no longer U7.RG1
- net N$28: now also U6.RG2; no longer U7.RG2
- net N$29: now also C17.1, U6.VOUT; no longer C21.1, U7.VOUT
- net N$3: now also C2.1; no longer C6.1
- net N$30: now also C17.2; no longer C21.2
- net N$31: now also U7.RG1; no longer U8.RG1
- net N$32: now also U7.RG2; no longer U8.RG2
- net N$34: now also C20.2; no longer C23.2
- net N$35: now also U8.RG1; no longer U9.RG1
- net N$36: now also U8.RG2; no longer U9.RG2
- net N$38: now also C23.2; no longer C25.2
- net N$39: now also U9.RG1; no longer U10.RG1
- net N$4: now also C2.2; no longer C6.2
- net N$40: now also U9.RG2; no longer U10.RG2
- net N$41: now also C26.1, U9.VOUT; no longer C27.1, U10.VOUT
- net N$42: now also C26.2; no longer C27.2
- net N$43: now also U14.XTAL1/CLKIN; no longer U11.XTAL1/CLKIN
- net N$44: now also C46.1, U14.CAP; no longer C28.1, U11.CAP
- net N$45: now also C44.2, U14.REFEXT; no longer C31.2, U11.REFEXT
- net N$46: now also U14.XTAL2; no longer U11.XTAL2
- net N$47: now also C45.2, U14.REFP; no longer C32.2, U11.REFP
- net N$48: now also U15.XTAL1/CLKIN; no longer U12.XTAL1/CLKIN
- net N$49: now also C51.1, U15.CAP; no longer C33.1, U12.CAP
- net N$5: now also JP2.2; no longer JP1.2
- net N$50: now also C49.2, U15.REFEXT; no longer C36.2, U12.REFEXT
- net N$51: now also U15.XTAL2; no longer U12.XTAL2
- net N$52: now also C50.2, U15.REFP; no longer C37.2, U12.REFP
- net N$53: now also U10.RG1; no longer U13.RG1
- net N$54: now also U10.RG2; no longer U13.RG2
- net N$55: now also C29.1, U10.VOUT; no longer C39.1, U13.VOUT
- net N$56: now also C29.2; no longer C39.2
- net N$57: now also U11.RG1; no longer U14.RG1
- net N$58: now also U11.RG2; no longer U14.RG2
- net N$59: now also C32.1, U11.VOUT; no longer C41.1, U14.VOUT
- net N$6: now also C41.1, U13.CAP; no longer C7.1, U3.CAP
- net N$60: now also C32.2; no longer C41.2
- net N$61: now also U12.RG1; no longer U15.RG1
- net N$62: now also U12.RG2; no longer U15.RG2
- net N$63: now also C35.1, U12.VOUT; no longer C43.1, U15.VOUT
- net N$64: now also C35.2; no longer C43.2
- net N$65: now also R45.2, U17.BOOT0; no longer R43.2, U16.BOOT0
- net N$66: now also R46.2, U17.NRST; no longer R44.2, U16.NRST
- net N$67: now also C53.2, R43.1, R44.2, U16.+IN; no longer C67.2, R45.2, R46.1, U17.+IN
- net N$7: now also U13.XTAL2; no longer U3.XTAL2
- net N$8: now also U13.XTAL1/CLKIN; no longer U3.XTAL1/CLKIN
- net N$9: now also C40.2, U13.REFP; no longer C8.2, U3.REFP
- net SWCLK: now also JP4.2, U17.PA14; no longer JP3.2, U16.PA14
- net SWDIO: now also JP4.3, U17.PA13; no longer JP3.3, U16.PA13
- net UART_RX: now also JP3.3, U17.PC11; no longer JP2.3, U16.PC11
- net UART_TX: now also JP3.2, U17.PC10; no longer JP2.2, U16.PC10
- net USB+: now also U17.PA12; no longer U16.PA12
- net USB-: now also U17.PA11; no longer U16.PA11
- net USB_ID: now also U17.PA10; no longer U16.PA10
Other:
- moved on the sheet: C1, C10, C11, C12, C13, C14, C15, C16, C17, C18, C19, C2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

Commit message: First Prototype Version of Schematic and PCB done
Parts:
- added C68, C69, C70, C71, C72, C73: 18p, rcl:C-EUC0603
- added J1: 12402012E212A, USB-C:12402012E212A
- added JP5, JP6: (no value), pinhead:PINHD-1X2
- added R53, R54: 5k1, rcl:R-EU_R0603
- added TP1, TP10, TP11, TP12, TP13, TP14, TP15, TP16, TP2, TP3, TP4, TP5, TP6, TP7, TP8, TP9: TPPAD1-17, testpad:TPPAD1-17
Connections:
- removed net ADC_CS: U13.!CS
- new net MCO: U17.PA8
- new net N$74: J1.CC1_A, R54.2
- new net N$75: J1.CC1_B, R53.1
- new net N$76: IC1.VO, JP5.2
- new net N$78: IC2.K, IC2.OUT, JP6.2
- net 2V5: now also TP16.TP
- net 3V3: now also JP6.1, TP3.TP; no longer C52.1, IC2.K, IC2.OUT, U16.V+
- net 5V: now also C25.1, C28.1, C31.1, C34.1, C52.1, JP5.1, TP2.TP, U16.V+; no longer IC1.VO
- net 9V: now also TP1.TP
- net ADC0: now also TP4.TP
- net ADC0_CS: now also U13.!CS
- net ADC1: now also TP5.TP
- net ADC10: now also TP14.TP
- net ADC11: now also TP15.TP
- net ADC2: now also TP6.TP
- net ADC3: now also TP7.TP
- net ADC4: now also TP8.TP
- net ADC5: now also TP9.TP
- net ADC6: now also TP10.TP
- net ADC7: now also TP11.TP
- net ADC8: now also TP12.TP
- net ADC9: now also TP13.TP
- net GND: now also C68.1, C69.1, C70.1, C71.1, C72.1, C73.1, J1.GND, J1.SHIELD, R53.2, R54.1
- net N$43: now also C69.2
- net N$46: now also C68.2
- net N$48: now also C70.2, U15.XTAL2, Y3.3; no longer U15.XTAL1/CLKIN, Y3.1
- net N$51: now also C71.2, U15.XTAL1/CLKIN, Y3.1; no longer U15.XTAL2, Y3.3
- net N$7: now also C72.2
- net N$8: now also C73.2
- net USB+: now also J1.D+_A, J1.D+_B
- net USB-: now also J1.D-_A, J1.D-_B
Other:
- moved on the sheet: C1, C10, C11, C12, C13, C14, C15, C16, C17, C18, C19, C2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
