File: Electronics/2024-03-01_Twin_Io.brd (EAGLE design)
At the start: 66.7 x 67.3 mm, 182 parts, among them IC1 7805, IC2 LD1117S33, J1 12402012E212A, U1 INA317IDGKT, U10 INA317IDGKT, U11 INA317IDGKT, U12 INA317IDGKT, U13 ADS131A04IPBSR, U14 ADS131A04IPBSR, U15 ADS131A04IPBSR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

Commit message: Final changes for V00-00-00
Parts:
- added R58, R59, R60, R61, R62, R63, R64, R65, R66, R67, R68, R69: 220k, rcl:R0603
- added S1, S4, S5: B3U-1000P, B3U-1000P:SW_B3U-1000P
- C12, C15, C18, C21, C24, C27, C3, C30, C33, C36, C6, C9: value 33nF/C0G -> 10nF/C0G
- R11, R14, R17, R2, R20, R23, R26, R29, R32, R35, R5, R8: value 10k -> 33k
Connections:
- new net N$77: R58.2, U1.3
- new net N$79: R59.2, U2.3
- new net N$80: R60.2, U3.3
- new net N$81: R61.2, U4.3
- new net N$82: R62.2, U5.3
- new net N$83: R63.2, U6.3
- new net N$84: R64.2, U7.3
- new net N$85: R65.2, U8.3
- new net N$86: R66.2, U9.3
- new net N$87: R67.2, U10.3
- new net N$88: R68.2, U11.3
- new net N$89: R69.2, U12.3
- new net SW0: S1.2, U17.3
- new net SW1: S4.2, U17.4
- new net SW2: S5.2, U17.5
- net GND: now also S1.1, S4.1, S5.1
- net LEAD0: now also R58.1; no longer U1.3
- net LEAD1: now also R59.1; no longer U2.3
- net LEAD10: now also R68.1; no longer U11.3
- net LEAD11: now also R69.1; no longer U12.3
- net LEAD2: now also R60.1; no longer U3.3
- net LEAD3: now also R61.1; no longer U4.3
- net LEAD4: now also R62.1; no longer U5.3
- net LEAD5: now also R63.1; no longer U6.3
- net LEAD6: now also R64.1; no longer U7.3
- net LEAD7: now also R65.1; no longer U8.3
- net LEAD8: now also R66.1; no longer U9.3
- net LEAD9: now also R67.1; no longer U10.3
Routing:
- net 2V5: track 211.7 -> 97.3 mm, vias 63 -> 40
- net N$89: track 0.00 -> 18.1 mm, vias 0 -> 1
- net LEAD11: track 20.0 -> 2.96 mm
- net N$77: track 0.00 -> 16.1 mm, vias 0 -> 1
- net LEAD0: track 18.8 -> 2.96 mm
- net LEAD10: track 18.6 -> 2.96 mm
- net N$88: track 0.00 -> 15.6 mm, vias 0 -> 1
- net LEAD1: track 17.7 -> 2.96 mm
- net N$79: track 0.00 -> 13.5 mm, vias 0 -> 1
- net SW2: track 0.00 -> 13.4 mm
- net LEAD9: track 16.1 -> 2.96 mm
- net N$87: track 0.00 -> 12.4 mm, vias 0 -> 1
- net SW1: track 0.00 -> 11.3 mm
- net LEAD2: track 14.2 -> 2.96 mm
- net SW0: track 0.00 -> 10.7 mm
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- added copper zone on layer 16, net 2V5
Other:
- board text added: "H0"
- board text added: "H1"
- board text added: "H2"
- board text added: "JLCJLCJLCJLC"
- board text added: "Pascal Bilger 03.03.2024"
- board text added: "SW0"
- board text added: "SW1"
- board text added: "SW2"
- board text removed: "By Pascal Bilger 03.03.2024"

Commit message: Changed the Resistors which connect the STM32 to the clock input of the ADC from 0R to 50R
Parts:
- R55, R56, R57: value 0R -> 50R
Changed lines of the file:
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@@
 <layers>
 <layer number="1" name="Top" color="4" fill="1" visible="yes" active="yes"/>
-<layer number="2" name="Route2" color="16" fill="1" visible="no" active="yes"/>
+<layer number="2" name="Route2" color="16" fill="1" visible="yes" active="yes"/>
 <layer number="3" name="Route3" color="17" fill="1" visible="no" active="no"/>
 <layer number="4" name="Route4" color="18" fill="1" visible="no" active="no"/>
@@
 <layer number="13" name="Route13" color="21" fill="1" visible="no" active="no"/>
 <layer number="14" name="Route14" color="22" fill="1" visible="no" active="no"/>
-<layer number="15" name="Route15" color="23" fill="1" visible="no" active="yes"/>
+<layer number="15" name="Route15" color="23" fill="1" visible="yes" active="yes"/>
 <layer number="16" name="Bottom" color="1" fill="1" visible="yes" active="yes"/>
 <layer number="17" name="Pads" color="2" fill="1" visible="yes" active="yes"/>
@@
 <layer number="20" name="Dimension" color="24" fill="1" visible="yes" active="yes"/>
 <layer number="21" name="tPlace" color="7" fill="1" visible="yes" active="yes"/>
-<layer number="22" name="bPlace" color="7" fill="1" visible="yes" active="yes"/>
+<layer number="22" name="bPlace" color="7" fill="1" visible="no" active="yes"/>
 <layer number="23" name="tOrigins" color="15" fill="1" visible="yes" active="yes"/>
 <layer number="24" name="bOrigins" color="15" fill="1" visible="yes" active="yes"/>
@@
 <hole x="50.8" y="75.565" drill="3.556"/>
 <text x="29.845" y="80.645" size="1.27" layer="22" rot="MR0">JLCJLCJLCJLC</text>
-<dimension x1="18.805" y1="77.175" x2="18.805" y2="76.525" x3="19.685" y3="76.85" textsize="1.778" layer="21"/>
 </plain>
 <attributes>
@@
 <attribute name="VALUE" x="64.77" y="44.45" size="1.27" layer="27" rot="R180"/>
 </element>
-<element name="R55" library="rcl" library_urn="urn:adsk.eagle:library:334" package="R0603" package3d_urn="urn:adsk.eagle:package:23555/3" value="0R" x="47.625" y="71.12" smashed="yes" rot="R180">
+<element name="R55" library="rcl" library_urn="urn:adsk.eagle:library:334" package="R0603" package3d_urn="urn:adsk.eagle:package:23555/3" value="50R" x="47.625" y="71.12" smashed="yes" rot="R180">
 <attribute name="NAME" x="48.26" y="70.485" size="1.27" layer="25" rot="R180"/>
 <attribute name="POPULARITY" value="70" x="47.625" y="71.12" size="1.778" layer="27" rot="R180" display="off"/>
@@
 <attribute name="VALUE" x="48.26" y="73.025" size="1.27" layer="27" rot="R180"/>
 </element>
-<element name="R56" library="rcl" library_urn="urn:adsk.eagle:library:334" package="R0603" package3d_urn="urn:adsk.eagle:package:23555/3" value="0R" x="50.8" y="50.165" smashed="yes" rot="R180">
+<element name="R56" library="rcl" library_urn="urn:adsk.eagle:library:334" package="R0603" package3d_urn="urn:adsk.eagle:package:23555/3" value="50R" x="50.8" y="50.165" smashed="yes" rot="R180">
 <attribute name="NAME" x="51.435" y="49.53" size="1.27" layer="25" rot="R180"/>
 <attribute name="POPULARITY" value="70" x="50.8" y="50.165" size="1.778" layer="27" rot="R180" display="off"/>
@@
 <attribute name="VALUE" x="51.435" y="52.07" size="1.27" layer="27" rot="R180"/>
 </element>
-<element name="R57" library="rcl" library_urn="urn:adsk.eagle:library:334" package="R0603" package3d_urn="urn:adsk.eagle:package:23555/3" value="0R" x="46.99" y="36.195" smashed="yes" rot="R270">
+<element name="R57" library="rcl" library_urn="urn:adsk.eagle:library:334" package="R0603" package3d_urn="urn:adsk.eagle:package:23555/3" value="50R" x="46.99" y="36.195" smashed="yes" rot="R270">
 <attribute name="NAME" x="47.625" y="36.83" size="1.27" layer="25" rot="R270"/>
 <attribute name="POPULARITY" value="70" x="46.99" y="36.195" size="1.778" layer="27" rot="R270" display="off"/>
