File: Electronics/2024-03-01_Twin_Io.sch (EAGLE design)
At the start: 182 parts, among them IC1 7805, IC2 LD1117S33, J1 12402012E212A, U1 INA317IDGKT, U10 INA317IDGKT, U11 INA317IDGKT, U12 INA317IDGKT, U13 ADS131A04IPBSR, U14 ADS131A04IPBSR, U15 ADS131A04IPBSR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

Commit message: Final changes for V00-00-00
Parts:
- added R58, R59, R60, R61, R62, R63, R64, R65, R66, R67, R68, R69: 220k, rcl:R-EU_R0603
- added S1, S4, S5: B3U-1000P, B3U-1000P:B3U-1000P
- C12, C15, C18, C21, C24, C27, C3, C30, C33, C36, C6, C9: value 33nF/C0G -> 10nF/C0G
- R11, R14, R17, R2, R20, R23, R26, R29, R32, R35, R5, R8: value 10k -> 33k
Connections:
- new net N$77: R58.2, U1.+
- new net N$79: R59.2, U2.+
- new net N$80: R60.2, U3.+
- new net N$81: R61.2, U4.+
- new net N$82: R62.2, U5.+
- new net N$83: R63.2, U6.+
- new net N$84: R64.2, U7.+
- new net N$85: R65.2, U8.+
- new net N$86: R66.2, U9.+
- new net N$87: R67.2, U10.+
- new net N$88: R68.2, U11.+
- new net N$89: R69.2, U12.+
- new net SW0: S1.2, U17.PC14-OSC32_IN
- new net SW1: S4.2, U17.PC15-OSC32_OUT
- new net SW2: S5.2, U17.PD0-OSC_IN
- net GND: now also S1.1, S4.1, S5.1
- net LEAD0: now also R58.1; no longer U1.+
- net LEAD1: now also R59.1; no longer U2.+
- net LEAD10: now also R68.1; no longer U11.+
- net LEAD11: now also R69.1; no longer U12.+
- net LEAD2: now also R60.1; no longer U3.+
- net LEAD3: now also R61.1; no longer U4.+
- net LEAD4: now also R62.1; no longer U5.+
- net LEAD5: now also R63.1; no longer U6.+
- net LEAD6: now also R64.1; no longer U7.+
- net LEAD7: now also R65.1; no longer U8.+
- net LEAD8: now also R66.1; no longer U9.+
- net LEAD9: now also R67.1; no longer U10.+
Other:
- note added: "If high pass filter is omitted assemble 0R resistor instead of C2"
- note removed: "If high pass filter is omitted assemble 0R resistor instead of C6"

Commit message: Changed the Resistors which connect the STM32 to the clock input of the ADC from 0R to 50R
Parts:
- R55, R56, R57: value 0R -> 50R
Changed lines of the file:
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@@
 <part name="JP5" library="pinhead" library_urn="urn:adsk.eagle:library:325" deviceset="PINHD-1X2" device="" package3d_urn="urn:adsk.eagle:package:22435/2"/>
 <part name="JP6" library="pinhead" library_urn="urn:adsk.eagle:library:325" deviceset="PINHD-1X2" device="" package3d_urn="urn:adsk.eagle:package:22435/2"/>
-<part name="R55" library="rcl" library_urn="urn:adsk.eagle:library:334" deviceset="R-EU_" device="R0603" package3d_urn="urn:adsk.eagle:package:23555/3" value="0R"/>
-<part name="R56" library="rcl" library_urn="urn:adsk.eagle:library:334" deviceset="R-EU_" device="R0603" package3d_urn="urn:adsk.eagle:package:23555/3" value="0R"/>
-<part name="R57" library="rcl" library_urn="urn:adsk.eagle:library:334" deviceset="R-EU_" device="R0603" package3d_urn="urn:adsk.eagle:package:23555/3" value="0R"/>
+<part name="R55" library="rcl" library_urn="urn:adsk.eagle:library:334" deviceset="R-EU_" device="R0603" package3d_urn="urn:adsk.eagle:package:23555/3" value="50R"/>
+<part name="R56" library="rcl" library_urn="urn:adsk.eagle:library:334" deviceset="R-EU_" device="R0603" package3d_urn="urn:adsk.eagle:package:23555/3" value="50R"/>
+<part name="R57" library="rcl" library_urn="urn:adsk.eagle:library:334" deviceset="R-EU_" device="R0603" package3d_urn="urn:adsk.eagle:package:23555/3" value="50R"/>
 <part name="R58" library="rcl" library_urn="urn:adsk.eagle:library:334" deviceset="R-EU_" device="R0603" package3d_urn="urn:adsk.eagle:package:23555/3" value="220k"/>
 <part name="R59" library="rcl" library_urn="urn:adsk.eagle:library:334" deviceset="R-EU_" device="R0603" package3d_urn="urn:adsk.eagle:package:23555/3" value="220k"/>
